Commit message: fix : hc_arm is not machin fixed and stl is found

File: catkin_ws/src/motoman_copy/motoman_hc10_support/urdf/hc10_macro.xacro (robot description, xacro)
@@ -73,5 +73,5 @@
       <collision>
         <geometry>
-          <mesh filename="package://motjoint_1_soman_hc10_support/meshes/hc10/collision/link_3_u.stl"/>
+          <mesh filename="package://motoman_hc10_support/meshes/hc10/collision/link_3_u.stl"/>
         </geometry>
       </collision>

Commit message: fix : removed redundant joint and regenerated urdf

File: catkin_ws/src/motoman_copy/motoman_hc10_support/urdf/hc10_macro.xacro (robot description, xacro)
@@ -193,10 +193,4 @@
     <!-- end of joint list -->
     <!-- ROS base_link to Robot Manufacturer World Coordinates transform -->
-    <link name="${prefix}base" />
-    <joint name="${prefix}base_link-base" type="fixed">
-      <origin xyz="0 0 0.275" rpy="0 0 0"/>
-      <parent link="${prefix}base_link"/>
-      <child link="${prefix}base"/>
-    </joint>
   </xacro:macro>
 </robot>

File: catkin_ws/src/motoman_copy/motoman_hc10_support/urdf/model_hc10.urdf (robot description, URDF)
Before this commit: robot motoman_hc10, 10 links, 9 joints
Links:
- removed link base
Joints:
- removed joint base_link-base
