Commit message: feat : added link between moveit and gazebo

File: catkin_ws/src/motoman_copy/motoman_hc10_support/urdf/hc10.control.xacro (robot description, xacro)
@@ -7,8 +7,8 @@
                 <type>transmission_interface/SimpleTransmission</type>
                 <joint name="${joint}">
-                    <hardwareInterface>hardware_interface/EffortJointInterface</hardwareInterface>
+                    <hardwareInterface>hardware_interface/PositionJointInterface</hardwareInterface>
                 </joint>
                 <actuator name="${motor}">
-                    <hardwareInterface>hardware_interface/EffortJointInterface</hardwareInterface>
+                    <hardwareInterface>hardware_interface/PositionJointInterface</hardwareInterface>
                     <mechanicalReduction>1</mechanicalReduction>
                 </actuator>
@@ -21,5 +21,4 @@
         <xacro:arm_control transmission="${arm_id}tran_5" joint="${arm_id}joint_5_b" motor="${arm_id}motor_5"/>
         <xacro:arm_control transmission="${arm_id}tran_6" joint="${arm_id}joint_6_t" motor="${arm_id}motor_6"/>
-        <xacro:arm_control transmission="${arm_id}tran_7" joint="${arm_id}joint_6_t-tool0" motor="${arm_id}motor_7"/>
         <gazebo>
             <plugin name="gazebo_ros_control" filename="libgazebo_ros_control.so"/>

File: catkin_ws/src/motoman_copy/motoman_hc10_support/urdf/hc10.gazebo.xacro (robot description, xacro)
@@ -10,5 +10,5 @@
             </gazebo>
         </xacro:macro>
-        <xacro:macro name="hand_gazebo" params="link">
+        <xacro:macro name="tool_gazebo" params="link">
             <gazebo reference="${link}">
                 <material>Gazebo/Grey</material>
@@ -24,5 +24,5 @@
         <xacro:arm_gazebo link="${arm_id}link_5_b"/>
         <xacro:arm_gazebo link="${arm_id}link_6_t"/>
-        <xacro:hand_gazebo link="${arm_id}tool0"/>
+        <xacro:tool_gazebo link="${arm_id}tool0"/>
     </xacro:macro>
 </robot>
