Commit message: feat: added moveit package
hc_10 arm is not a chain error still written WIP

File: catkin_ws/src/motoman_copy/motoman_hc10_support/urdf/hc10.xacro (robot description, xacro)
@@ -3,3 +3,7 @@
   <xacro:include filename="$(find motoman_hc10_support)/urdf/hc10_macro.xacro" />
   <xacro:motoman_hc10 prefix=""/>
+  <xacro:include filename="$(find motoman_hc10_support)/urdf/hc10.gazebo.xacro"/>
+  <xacro:hc10_gazebo arm_id=""/>
+  <xacro:include filename="$(find motoman_hc10_support)/urdf/hc10.control.xacro"/>
+  <xacro:hc10_control arm_id=""/>
 </robot>

File: catkin_ws/src/motoman_copy/motoman_hc10_support/urdf/hc10_macro.xacro (robot description, xacro)
@@ -73,5 +73,5 @@
       <collision>
         <geometry>
-          <mesh filename="package://motoman_hc10_support/meshes/hc10/collision/link_3_u.stl"/>
+          <mesh filename="package://motjoint_1_soman_hc10_support/meshes/hc10/collision/link_3_u.stl"/>
         </geometry>
       </collision>

Commit message: add kinect sensor, gazebo & rviz OK

File: catkin_ws/src/motoman_copy/motoman_hc10_support/urdf/hc10.xacro (robot description, xacro)
@@ -7,3 +7,5 @@
   <xacro:include filename="$(find motoman_hc10_support)/urdf/hc10.control.xacro"/>
   <xacro:hc10_control arm_id=""/>
+  <xacro:include filename="$(find motoman_hc10_support)/urdf/kinect_macro.xacro" />
+  <xacro:motoman_hc10_kinect prefix=""/>
 </robot>

File: catkin_ws/src/motoman_copy/motoman_hc10_support/urdf/model_hc10.urdf (robot description, URDF)
Before this commit: robot motoman_hc10, 9 links, 8 joints
Links:
- added link camera_depth_frame, mass 0.1; visual mesh filename=package://motoman_hc10_support/meshes/hc10/visual/kinect.dae
- added link camera_depth_optical_frame
Joints:
- added joint cam_t_optical: type fixed, parent camera_depth_frame, child camera_depth_optical_frame, origin xyz=0 0 0 rpy= -1.5707963267948966 0 -1.5707963267948966
- added joint tool0_t_cam: type fixed, parent tool0, child camera_depth_frame, origin xyz=0 -0.06 0.05 rpy=0 -1.5707963267948966 -1.5707963267948966
